Commit message: updated fred by making all links 1 unit

File: fredFP.urdf (robot description, URDF)
Before this commit: robot Fred, 10 links, 9 joints
Links:
- link FLLL: geometry collision box size=1 0.15 0.15; visual box size=1 0.15 0.15
- link FLUL: geometry collision box size=1 0.2 0.2; visual box size=1 0.2 0.2
- link FRLL: geometry collision box size=1 0.15 0.15; visual box size=1 0.15 0.15
- link FRUL: geometry collision box size=1 0.2 0.2; visual box size=1 0.2 0.2
- link RLLL: geometry collision box size=1 0.15 0.15; visual box size=1 0.15 0.15
- link RLUL: geometry collision box size=1 0.2 0.2; visual box size=1 0.2 0.2
- link RRLL: geometry collision box size=1 0.15 0.15; visual box size=1 0.15 0.15
- link RRUL: geometry collision box size=1 0.2 0.2; visual box size=1 0.2 0.2
Joints:
- joint FLelbow: origin xyz=0 .175 -1 -> xyz=0 .175 -0.9
- joint FRelbow: origin xyz=0 -.175 -1 -> xyz=0 -.175 -0.9
- joint RLelbow: origin xyz=0 .175 -1 -> xyz=0 .175 -0.9
- joint RRelbow: origin xyz=0 -.175 -1 -> xyz=0 -.175 -0.9

Commit message: Update fredFP.urdf

File: fredFP.urdf (robot description, URDF)
Before this commit: robot Fred, 10 links, 9 joints
Links:
- link camera: mass 0.1 -> None
Joints:
- joint FLelbow: type continuous -> revolute
- joint FLshoulder: type continuous -> revolute
- joint FRelbow: type continuous -> revolute
- joint FRhoulder: type continuous -> revolute
- joint RLelbow: type continuous -> revolute
- joint RLshoulder: type continuous -> revolute
- joint RRelbow: type continuous -> revolute
- joint RRshoulder: type continuous -> revolute

Commit message: Add files via upload

File: fredFP.urdf (robot description, URDF)
Before this commit: robot Fred, 10 links, 9 joints
Links:
- link camera: mass None -> 0.1
Joints:
- joint FLelbow: type revolute -> continuous
- joint FLshoulder: type revolute -> continuous
- joint FRelbow: type revolute -> continuous
- joint FRhoulder: type revolute -> continuous
- joint RLelbow: type revolute -> continuous
- joint RLshoulder: type revolute -> continuous
- joint RRelbow: type revolute -> continuous
- joint RRshoulder: type revolute -> continuous
